File: PowerSeparate/Digital.kicad_sch (KiCad schematic)
At the start: 10 parts, among them J4 D_Power, J5 D_Power, J6 D_Power

Commit message: MC2
ガーバーデータ出力
BOMファイル出力
NJM2374A関連プロジェクトを作成
PowerSeparateが完了
Connections:
- net D+5V is gone; now on net +5VD: PwC3.1, PwL1.2
- net GNDD is gone; now on net GND: PwC1.2, PwC2.2, PwC3.2, PwIC1.2 (GND), PwJ4.2 (Pin_2)
