File: VCFSeparate/VCFSeparate.kicad_pcb (KiCad board)
At the start: 2 copper layers, 100 x 75 mm, 82 parts, among them J1 A_Power, J2 Input, J3 AudioOut, Q1 Q_PNP_ECB, Q2 Q_PNP_ECB, Q3 Q_PNP_ECB, Q4 Q_PNP_ECB, U1 LM13700, U2 LM13700, U3 LM13700, U4 Opamp_Dual, U5 Opamp_Dual, U6 Opamp_Dual, U7 Opamp_Dual

Commit message: MC2
ここまででFIXした内容
Parts:
- J2: footprint Connector_PinSocket_2.54mm:PinSocket_2x05_P2.54mm_Vertical -> Connector_PinSocket_2.54mm:PinSocket_2x06_P2.54mm_Vertical
- VR1: footprint SamacSys_Parts:3296W1502A -> SamacSys_parts:3296W1502A
- VR2, VR3, VR4, VR5, VR6, VR7: footprint SamacSys_Parts:RK09D117000B -> SamacSys_parts:RK09D117000B
- moved J2 2.63 mm to (64.9, 79.2)
Connections:
- J2 pad 10: GNDA -> VCAEnv
- J2 pad 3: Env -> FilterEnv
- J2 pad 4: Env -> FilterEnv
- J2 pad 9: GNDA -> VCAEnv
- R44 pad 1: Env -> VCAEnv
- VR3 pad 1: Env -> FilterEnv
Routing:
- net Env: track 97.5 -> 0.00 mm, vias 1 -> 0
- net VCAEnv: track 0.00 -> 79.9 mm, vias 0 -> 2
- net FilterEnv: track 0.00 -> 63.7 mm, vias 0 -> 1
- net CV: track 107.9 -> 99.5 mm
- net LFOSine: track 70.3 -> 74.0 mm, vias 2 -> 1
- net VCF_IN: track 21.2 -> 23.9 mm
- net +5VA: track 111.9 -> 113.5 mm, vias 1 -> 3
Other:
- board text added: "FilterEnv"
- board text added: "MC2 VCF+VCA Separate Borad Rev1 2025/7/27"
- board text added: "VCAEnv"
- board text removed: "MC2 VCF+VCA Separate Borad 2025/6/24"
