File: VCFSeparate/CVMixer.kicad_sch (KiCad schematic)
At the start: 24 parts, among them J2 Input, Q1 Q_PNP_ECB, Q2 Q_PNP_ECB, Q3 Q_PNP_ECB, U4 Opamp_Dual, U5 Opamp_Dual

Commit message: MC2
デバッグ一通り完了して動作出来た
Parts:
- R26: value 56K -> 39K
- R29: value 280K -> 150K
Connections:
- net GNDA: now also Q1.2 (C); no longer Q1.1 (E)
- net at R28.1, R29.1: now also Q1.1 (E); no longer Q1.2 (C)
Changed lines of the file:
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@@
 	)
 	(junction
-		(at 109.22 114.3)
-		(diameter 0)
-		(color 0 0 0 0)
-	)
-	(junction
 		(at 81.28 149.86)
 		(diameter 0)
@@
 	)
 	(junction
+		(at 109.22 114.3)
+		(diameter 0)
+		(color 0 0 0 0)
+	)
+	(junction
 		(at 204.47 135.89)
 		(diameter 0)
@@
 	(wire
 		(pts
+			(xy 96.52 120.65) (xy 101.6 120.65)
+		)
+		(stroke
+			(width 0)
+			(type default)
+		)
+	)
+	(wire
+		(pts
 			(xy 139.7 63.5) (xy 129.54 63.5)
 		)
@@
 	(wire
 		(pts
+			(xy 109.22 114.3) (xy 109.22 115.57)
+		)
+		(stroke
+			(width 0)
+			(type default)
+		)
+	)
+	(wire
+		(pts
 			(xy 151.13 152.4) (xy 154.94 152.4)
 		)
@@
 	(wire
 		(pts
+			(xy 109.22 125.73) (xy 109.22 129.54)
+		)
+		(stroke
+			(width 0)
+			(type default)
+		)
+	)
+	(wire
+		(pts
 			(xy 109.22 113.03) (xy 109.22 114.3)
 		)
@@
 	(wire
 		(pts
-			(xy 109.22 114.3) (xy 109.22 115.57)
-		)
-		(stroke
-			(width 0)
-			(type default)
-		)
-	)
-	(wire
-		(pts
 			(xy 110.49 34.29) (xy 114.3 34.29)
 		)
@@
 	(wire
 		(pts
-			(xy 101.6 120.65) (xy 96.52 120.65)
-		)
-		(stroke
-			(width 0)
-			(type default)
-		)
-	)
-	(wire
-		(pts
 			(xy 81.28 73.66) (xy 77.47 73.66)
 		)
@@
 			)
 		)
-		(property "Value" "56K"
+		(property "Value" "39K"
 			(at 118.11 73.66 90)
 			(effects
@@
 	(symbol
 		(lib_id "power:GNDA")
-		(at 109.22 125.73 0)
+		(at 109.22 129.54 0)
 		(unit 1)
 		(exclude_from_sim no)
@@
 		(fields_autoplaced yes)
 		(property "Reference" "#PWR034"
-			(at 109.22 132.08 0)
+			(at 109.22 135.89 0)
 			(effects
 				(font
@@
 		)
 		(property "Value" "GNDA"
-			(at 109.22 130.81 0)
+			(at 109.22 134.62 0)
 			(effects
 				(font
@@
 		)
 		(property "Footprint" ""
-			(at 109.22 125.73 0)
+			(at 109.22 129.54 0)
 			(effects
 				(font
@@
 		)
 		(property "Datasheet" ""
-			(at 109.22 125.73 0)
+			(at 109.22 129.54 0)
 			(effects
 				(font
@@
 		)
 		(property "Description" "Power symbol creates a global label with name \"GNDA\" , analog ground"
-			(at 109.22 125.73 0)
+			(at 109.22 129.54 0)
 			(effects
 				(font
@@
 		(lib_id "Device:Q_PNP_ECB")
 		(at 106.68 120.65 0)
+		(mirror x)
 		(unit 1)
 		(exclude_from_sim no)
@@
 		(on_board yes)
 		(dnp no)
-		(fields_autoplaced yes)
 		(property "Reference" "Q1"
-			(at 111.76 119.3799 0)
+			(at 112.522 119.888 0)
 			(effects
 				(font
@@
 		)
 		(property "Value" "Q_PNP_ECB"
-			(at 111.76 121.9199 0)
+			(at 112.522 121.92 0)
 			(effects
 				(font
@@
 		)
 		(property "Footprint" "Package_TO_SOT_THT:TO-92_HandSolder"
-			(at 111.76 118.11 0)
+			(at 111.76 123.19 0)
 			(effects
 				(font
@@
 			)
 		)
-		(property "Value" "280K"
+		(property "Value" "150K"
 			(at 118.11 111.76 90)
 			(effects
