File: VCOSeparate/VCO.kicad_sch (KiCad schematic)
At the start: 47 parts, among them IC1 V3340M, IC2 AS321KTR-E1

Commit message: MC2
ここまででFIXした内容
Parts:
- added C48: 0.01uF, Capacitor_THT:C_Disc_D5.0mm_W2.5mm_P2.50mm, symbol Device:C
- added R113: 560, Resistor_THT:R_Axial_DIN0207_L6.3mm_D2.5mm_P2.54mm_Vertical, symbol Device:R
- IC1: footprint DIP794W56P260L1905H432Q16N -> SamacSys_parts:DIP794W56P260L1905H432Q16N
- IC2: footprint SOT95P282X145-5N -> SamacSys_parts:SOT95P282X145-5N
- S1: footprint ASLB1470 -> SamacSys_parts:ASLB1470
- S2: footprint OS103011MS8QP1 -> SamacSys_parts:OS103011MS8QP1
- VR3, VR4, VR6: footprint SamacSys_Parts:RK09D117000B -> SamacSys_parts:RK09D117000B
Connections:
- net GNDA: now also C48.1
- net Vfci: now also R113.1
- new net: C48.2, R113.2
Other:
- moved on the sheet: R104, VR4

Commit message: MC2
デバッグ一通り完了して動作出来た
Parts:
- removed S1: ASLB1470, SamacSys_parts:ASLB1470, symbol SamacSys_Parts:ASLB1470
- added C2: 0.01uF, Capacitor_THT:C_Disc_D5.0mm_W2.5mm_P2.50mm, symbol Device:C
- added R4: 1M, Resistor_THT:R_Axial_DIN0207_L6.3mm_D2.5mm_P2.54mm_Vertical, symbol Device:R
- added S4: SS14D0839VG5PA, SS14D0839VG5PA, symbol SamacSys_Parts:SS14D0839VG5PA
- R1: value 100K -> 10K
Connections:
- net GNDA: now also S4.MH1, S4.MH2; no longer C51.1, C52.1
- net at R41.2, R42.1: now also S4.1
- net at R40.2, R41.1: now also S4.2
- net at R39.2, R40.1: now also S4.4
- net at R38.2, R39.1: now also S4.5
- net at IC2.1 (INPUT_+): now also S4.3
- net at IC1.13, R119.1, R127.1: now also R4.1
- net Vtri: now reaches IC1.10
- new net: C2.2, R4.2
- new net HardSyncIn: C51.1
- new net LFM_In: C2.1
- new net SoftSyncIn: C52.1
- no-connect marks 2 -> 0
Other:
- moved on the sheet: C55, R127
