File: debugVCASeparate/VCA.kicad_sch (KiCad schematic)
At the start: 30 parts, among them J2 AudioIn, J3 AudioOut, J4 VCAEnv, Q2 Q_PNP_ECB, U2 LM13700, U3 Opamp_Dual, U4 Opamp_Dual

Commit message: MC2
デバッグ一通り完了して動作出来た
Parts:
- removed J2: AudioIn, Connector_PinSocket_2.54mm:PinSocket_1x03_P2.54mm_Vertical, symbol Connector_Generic:Conn_01x03
- added J2: AudioIn, Connector_PinSocket_2.54mm:PinSocket_1x02_P2.54mm_Vertical, symbol Connector_Generic:Conn_01x02
Connections:
- net GNDA: now also J2.2 (Pin_2)
- net VCF_OUT: now also J2.1 (Pin_1)
- net ResoWav renamed VCA_ResoWav
Changed lines of the file:
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@@
 	(wire
 		(pts
-			(xy 62.23 36.83) (xy 59.69 36.83)
+			(xy 64.77 34.29) (xy 59.69 34.29)
 		)
 		(stroke
@@
 	(wire
 		(pts
+			(xy 60.96 31.75) (xy 64.77 31.75)
+		)
+		(stroke
+			(width 0)
+			(type default)
+		)
+	)
+	(wire
+		(pts
 			(xy 156.21 86.36) (xy 156.21 78.74)
 		)
@@
 	(wire
 		(pts
-			(xy 59.69 36.83) (xy 59.69 39.37)
+			(xy 59.69 34.29) (xy 59.69 39.37)
 		)
 		(stroke
@@
 		)
 	)
-	(global_label "VCAEnv"
-		(shape input)
-		(at 34.29 129.54 180)
+	(global_label "VCF_OUT"
+		(shape output)
+		(at 60.96 31.75 180)
 		(fields_autoplaced yes)
 		(effects
@@
 		)
 		(property "Intersheetrefs" "${INTERSHEET_REFS}"
-			(at 28.0392 129.54 0)
+			(at 49.9314 31.75 0)
 			(effects
 				(font
@@
 		)
 	)
-	(global_label "VCF_OUT"
+	(global_label "VCAEnv"
 		(shape input)
-		(at 27.94 73.66 180)
+		(at 34.29 129.54 180)
 		(fields_autoplaced yes)
 		(effects
@@
 		)
 		(property "Intersheetrefs" "${INTERSHEET_REFS}"
-			(at 16.9114 73.66 0)
+			(at 28.0392 129.54 0)
 			(effects
 				(font
@@
 		)
 	)
-	(global_label "ResoWav"
+	(global_label "VCF_OUT"
 		(shape input)
-		(at 27.94 62.23 180)
+		(at 27.94 73.66 180)
 		(fields_autoplaced yes)
 		(effects
@@
 		)
 		(property "Intersheetrefs" "${INTERSHEET_REFS}"
-			(at 16.8511 62.23 0)
+			(at 16.9114 73.66 0)
 			(effects
 				(font
@@
 		)
 	)
-	(global_label "VCACnt"
-		(shape output)
-		(at 166.37 139.7 0)
+	(global_label "VCA_ResoWav"
+		(shape input)
+		(at 27.94 62.23 180)
 		(fields_autoplaced yes)
 		(effects
@@
 				(size 1.27 1.27)
 			)
-			(justify left)
+			(justify right)
 		)
 		(property "Intersheetrefs" "${INTERSHEET_REFS}"
-			(at 175.9471 139.7 0)
+			(at 12.4363 62.23 0)
 			(effects
 				(font
 					(size 1.27 1.27)
 				)
-				(justify left)
+				(justify right)
 				(hide yes)
 			)
 		)
 	)
-	(global_label "VCF_OUT"
+	(global_label "VCACnt"
 		(shape output)
-		(at 62.23 34.29 180)
+		(at 166.37 139.7 0)
 		(fields_autoplaced yes)
 		(effects
@@
 				(size 1.27 1.27)
 			)
-			(justify right)
+			(justify left)
 		)
 		(property "Intersheetrefs" "${INTERSHEET_REFS}"
-			(at 51.2014 34.29 0)
+			(at 175.9471 139.7 0)
 			(effects
 				(font
 					(size 1.27 1.27)
 				)
-				(justify right)
+				(justify left)
 				(hide yes)
 			)
@@
 		)
 	)
-	(global_label "ResoWav"
-		(shape output)
-		(at 62.23 31.75 180)
-		(fields_autoplaced yes)
-		(effects
-			(font
-				(size 1.27 1.27)
-			)
-			(justify right)
-		)
-		(property "Intersheetrefs" "${INTERSHEET_REFS}"
-			(at 51.1411 31.75 0)
-			(effects
-				(font
-					(size 1.27 1.27)
-				)
-				(justify right)
-				(hide yes)
-			)
-		)
-	)
 	(symbol
 		(lib_id "Device:R")
@@
 	)
 	(symbol
+		(lib_id "Connector_Generic:Conn_01x02")
+		(at 69.85 31.75 0)
+		(unit 1)
+		(exclude_from_sim no)
+		(in_bom yes)
+		(on_board yes)
+		(dnp no)
+		(fields_autoplaced yes)
+		(property "Reference" "J2"
+			(at 72.39 31.7499 0)
+			(effects
+				(font
+					(size 1.27 1.27)
+				)
+				(justify left)
+			)
+		)
+		(property "Value" "AudioIn"
+			(at 72.39 34.2899 0)
+			(effects
+				(font
+					(size 1.27 1.27)
+				)
+				(justify left)
+			)
+		)
+		(property "Footprint" "Connector_PinSocket_2.54mm:PinSocket_1x02_P2.54mm_Vertical"
+			(at 69.85 31.75 0)
+			(effects
+				(font
+					(size 1.27 1.27)
+				)
+				(hide yes)
+			)
+		)
+		(property "Datasheet" "~"
+			(at 69.85 31.75 0)
+			(effects
+				(font
+					(size 1.27 1.27)
+				)
+				(hide yes)
+			)
+		)
+		(property "Description" "Generic connector, single row, 01x02, script generated (kicad-library-utils/schlib/autogen/connector/)"
+			(at 69.85 31.75 0)
+			(effects
+				(font
+					(size 1.27 1.27)
+				)
+				(hide yes)
+			)
+		)
+		(pin "1"
+		)
+		(pin "2"
+		)
+		(instances
+			(project "debugVCASeparate"
+				(path "/20da34b0-f9e2-4ef1-be70-e6e2cca721c0/95ec37ca-e16f-40ae-99aa-b5e8d93e3c51"
+					(reference "J2")
+					(unit 1)
+				)
+			)
+		)
+	)
+	(symbol
 		(lib_id "power:GNDA")
 		(at 93.98 39.37 0)
@@
 					(unit 1)
 				)
-			)
-		)
-	)
-	(symbol
-		(lib_id "Connector_Generic:Conn_01x03")
-		(at 67.31 34.29 0)
-		(unit 1)
-		(exclude_from_sim no)
-		(in_bom yes)
-		(on_board yes)
-		(dnp no)
-		(fields_autoplaced yes)
-		(property "Reference" "J2"
-			(at 69.85 33.0199 0)
-			(effects
-				(font
-					(size 1.27 1.27)
-				)
-				(justify left)
-			)
-		)
-		(property "Value" "AudioIn"
-			(at 69.85 35.5599 0)
-			(effects
-				(font
-					(size 1.27 1.27)
-				)
-				(justify left)
-			)
-		)
-		(property "Footprint" "Connector_PinSocket_2.54mm:PinSocket_1x03_P2.54mm_Vertical"
-			(at 67.31 34.29 0)
-			(effects
-				(font
-					(size 1.27 1.27)
-				)
-				(hide yes)
-			)
-		)
-		(property "Datasheet" "~"
-			(at 67.31 34.29 0)
-			(effects
-				(font
-					(size 1.27 1.27)
-				)
-				(hide yes)
-			)
-		)
-		(property "Description" "Generic connector, single row, 01x03, script generated (kicad-library-utils/schlib/autogen/connector/)"
-			(at 67.31 34.29 0)
-			(effects
-				(font
-					(size 1.27 1.27)
-				)
-				(hide yes)
-			)
-		)
-		(pin "3"
-		)
-		(pin "2"
-		)
-		(pin "1"
-		)
-		(instances
-			(project ""
-				(path "/20da34b0-f9e2-4ef1-be70-e6e2cca721c0/95ec37ca-e16f-40ae-99aa-b5e8d93e3c51"
-					(reference "J2")
-					(unit 1)
-				)
