File: debugVCASeparate/VCF.kicad_sch (KiCad schematic)
At the start: 16 parts, among them Q1 Q_PNP_ECB, U1 Opamp_Dual, U2 LM13700

Commit message: MC2
デバッグ一通り完了して動作出来た
Parts:
- added J6: VCF_ResoWav, Connector_PinSocket_2.54mm:PinSocket_1x02_P2.54mm_Vertical, symbol Connector_Generic:Conn_01x02
- added R6, R7, R8: 10K, Resistor_THT:R_Axial_DIN0204_L3.6mm_D1.6mm_P7.62mm_Horizontal, symbol Device:R
- added R9: 1K, Resistor_THT:R_Axial_DIN0204_L3.6mm_D1.6mm_P7.62mm_Horizontal, symbol Device:R
- added U5: Opamp_Dual, Package_DIP:DIP-8_W7.62mm_Socket_LongPads, symbol Device:Opamp_Dual
- added VR1, VR2: 3362P 10K, SamacSys_parts:3362P_1, symbol SamacSys_Parts:3362P-1-103LF
Connections:
- net GNDA: now also J6.2 (Pin_2), R6.1, R8.1
- net ResoWav: no longer names the net of R23.2, U2.8
- net ResoWav: now also U5.3 (+), U5.5 (+)
- new net: R6.2, U5.2 (-), VR1.1 (CCW)
- new net: R8.2, U5.6 (-), VR2.1 (CCW)
- new net: R9.1, VR2.2 (WIPER), VR2.3 (CW)
- new net: R7.1, VR1.2 (WIPER), VR1.3 (CW)
- new net VCA_ResoWav: R9.2, U5.7
- new net VCF_ResoWav: J6.1 (Pin_1), R7.2, U5.1
Other:
- moved on the sheet: Q1, R11, R12, R13, R14, R15, R41, R43, U1A, U1B, VR6
