File: debugVCASeparate/VCF_VCA_Power.kicad_sch (KiCad schematic)
At the start: 6 parts, among them J1 A_Power, J5 A_Power, U1 Opamp_Dual, U2 LM13700, U3 Opamp_Dual, U4 Opamp_Dual

Commit message: MC2
デバッグ一通り完了して動作出来た
Parts:
- added U5: Opamp_Dual, Package_DIP:DIP-8_W7.62mm_Socket_LongPads, symbol Device:Opamp_Dual
Connections:
- net +12VA: now also U5.8 (V+)
- net -12VA: now also U5.4 (V-)
