File: debugVCASeparate/debugVCASeparate.kicad_pcb (KiCad board)
At the start: 2 copper layers, 80 x 70 mm, 47 parts, among them J1 A_Power, J2 AudioIn, J3 AudioOut, J4 VCAEnv, J5 A_Power, Q1 Q_PNP_ECB, Q2 Q_PNP_ECB, U1 Opamp_Dual, U2 LM13700, U3 Opamp_Dual, U4 Opamp_Dual

Commit message: MC2
デバッグ一通り完了して動作出来た
Parts:
- added J6: VCF_ResoWav, Connector_PinSocket_2.54mm:PinSocket_1x02_P2.54mm_Vertical, F.Cu at (50.8, 131.4)
- added R6: 10K, Resistor_THT:R_Axial_DIN0204_L3.6mm_D1.6mm_P7.62mm_Horizontal, F.Cu at (61.8, 113.2)
- added R7: 10K, Resistor_THT:R_Axial_DIN0204_L3.6mm_D1.6mm_P7.62mm_Horizontal, F.Cu at (61.8, 110.9)
- added R8: 10K, Resistor_THT:R_Axial_DIN0204_L3.6mm_D1.6mm_P7.62mm_Horizontal, F.Cu at (90.6, 112.9)
- added R9: 1K, Resistor_THT:R_Axial_DIN0204_L3.6mm_D1.6mm_P7.62mm_Horizontal, F.Cu at (90.6, 110.6)
- added U5: Opamp_Dual, Package_DIP:DIP-8_W7.62mm_Socket_LongPads, F.Cu at (72.1, 110.6)
- added VR1: 3362P 10K, SamacSys_parts:3362P_1, F.Cu at (65.5, 114.6)
- added VR2: 3362P 10K, SamacSys_parts:3362P_1, F.Cu at (85.5, 121.4)
- J2: footprint Connector_PinSocket_2.54mm:PinSocket_1x03_P2.54mm_Vertical -> Connector_PinSocket_2.54mm:PinSocket_1x02_P2.54mm_Vertical
- moved U4 14.6 mm to (84.6, 130.8)
- moved R47 14.6 mm to (81.7, 130.8)
- moved C7 14.6 mm to (81.4, 125.5)
- moved R48 14.6 mm to (81.7, 133.3)
- moved R49 14.6 mm to (84.5, 141.6)
- moved R38 14.6 mm to (74.0, 135.9)
- moved C9 14.4 mm to (91.5, 125.5)
- moved VR7 10.5 mm to (102.3, 138.3)
- moved VR6 10.4 mm to (59.5, 138.4)
- moved J1 7.37 mm to (48.8, 79.0)
- moved J5 7.37 mm to (48.8, 74.4)
- moved J4 5.61 mm to (112.0, 96.7), turned to 0 degrees
- moved J3 2.96 mm to (112.0, 106.3)
- moved J2 2.47 mm to (84.5, 72.9)
Connections:
- C1 pad 1: ResoWav -> VCA_ResoWav
- J2 pad 1: ResoWav -> VCF_OUT
- J2 pad 2: VCF_OUT -> GNDA
- R23 pad 2: ResoWav -> Net-(U5A-+)
- U2 pad 8: ResoWav -> Net-(U5A-+)
Routing:
- net ResoWav: track 51.1 -> 0.00 mm, vias 1 -> 0
- net VCA_ResoWav: track 0.00 -> 43.8 mm
- net VCF_ResoWav: track 0.00 -> 39.6 mm, vias 0 -> 1
- net Net-(U5A-+): track 0.00 -> 34.4 mm
- net -12VA: track 123.3 -> 144.4 mm
- net Net-(C7-Pad2): track 8.53 -> 23.6 mm
- net +5VA: track 55.6 -> 68.2 mm
- net Net-(VR1-CW): track 0.00 -> 11.4 mm
- net Net-(VR2-CW): track 0.00 -> 10.8 mm
- net Net-(Q2-E): track 17.8 -> 28.2 mm
- net Net-(VR6-WIPER): track 14.9 -> 24.7 mm
- net Net-(J3-Pin_1): track 25.6 -> 35.1 mm
- net Net-(U5B--): track 0.00 -> 9.45 mm
- net Net-(U5A--): track 0.00 -> 8.17 mm
- net Net-(VR7-CCW): track 25.7 -> 29.8 mm
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Other:
- board size 80 x 70 mm -> 80 x 79 mm
- board text added: "Audio Out"
- board text added: "VCA Env"
- board text added: "VCF ResoWav"
- board text added: "debugVCASeparate Rev2 2025/8/31"
- board text removed: "Reso Wave"
- board text removed: "debugVCASeparate 2025/8/11"
