File: debugVCFSeparate/CVMixer.kicad_sch (KiCad schematic)
At the start: 22 parts, among them J2 Input, Q1 Q_PNP_ECB, Q2 Q_PNP_ECB, Q4 Q_NPN_ECB, U3 Opamp_Dual

Commit message: MC2
デバッグ一通り完了して動作出来た
Parts:
- removed RV1: 100K, Potentiometer_THT:Potentiometer_Bourns_3386F_Vertical, symbol Device:R_Potentiometer_Trim
- added RV1: 3362P 100K, Potentiometer_THT:Potentiometer_Bourns_3386P_Vertical, symbol Device:R_Potentiometer_Trim_US
- R26: value 56K -> 39K
- R29: value 280K -> 150K
- VR1, VR2, VR4: value RK09D117000B -> 100KB
- VR3: value RK09D117000B -> 100KA
Connections:
- net +12VA: now also RV1.1
- net -12VA: now also RV1.3
- net GNDA: now also Q1.2 (C), U3.5 (+); no longer Q1.1 (E), U3.6 (-)
- net at R28.1, R29.1: now also Q1.1 (E); no longer Q1.2 (C)
- net at R25.2, R26.2, R27.2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: now also U3.6 (-); no longer U3.5 (+)
- net at R22.1: now also RV1.2
