File: debugVCFSeparate/debugVCFSeparate.kicad_pcb (KiCad board)
At the start: 2 copper layers, 90 x 79 mm, 54 parts, among them J1 A_Power, J2 Input, J3 InResoWav, J4 FltOrder, J5 VCFOut, Q1 Q_PNP_ECB, Q2 Q_PNP_ECB, Q4 Q_NPN_ECB, U1 LM13700, U2 LM13700, U3 Opamp_Dual

Commit message: MC2
デバッグ一通り完了して動作出来た
Parts:
- R26: value 56K -> 39K
- R29: value 280K -> 150K
- RV1: value 100K -> 3362P 100K; footprint Potentiometer_THT:Potentiometer_Bourns_3386F_Vertical -> Potentiometer_THT:Potentiometer_Bourns_3386P_Vertical
- VR1, VR2, VR4: value RK09D117000B -> 100KB
- VR3: value RK09D117000B -> 100KA
- moved C2 4.55 mm to (131.6, 93.7), turned to -90 degrees
- moved RV1 2.73 mm to (144.9, 62.4)
- moved Q1 2.67 mm to (177.8, 47.1), turned to 90 degrees
- moved R6 2.35 mm to (141.4, 88.8)
Connections:
- Q1 pad 1: GNDA -> Net-(Q1-E)
- Q1 pad 2: Net-(Q1-C) -> GNDA
- R25 pad 2: Net-(U3B-+) -> Net-(U3B--)
- R26 pad 2: Net-(U3B-+) -> Net-(U3B--)
- R27 pad 2: Net-(U3B-+) -> Net-(U3B--)
- R28 pad 1: Net-(Q1-C) -> Net-(Q1-E)
- R29 pad 1: Net-(Q1-C) -> Net-(Q1-E)
- R29 pad 2: Net-(U3B-+) -> Net-(U3B--)
- R39 pad 1: Net-(U3B-+) -> Net-(U3B--)
- U3 pad 5: Net-(U3B-+) -> GNDA
- U3 pad 6: GNDA -> Net-(U3B--)
Routing:
- net Net-(U3B-+): track 59.1 -> 0.00 mm, vias 1 -> 0
- net Net-(U3B--): track 0.00 -> 58.4 mm
- net +12VA: track 107.5 -> 128.7 mm
- net Net-(Q1-C): track 12.8 -> 0.00 mm
- net Net-(Q1-E): track 0.00 -> 9.71 mm
- net LFOSine: track 42.8 -> 50.5 mm
- net LP12db: track 39.6 -> 45.7 mm
- net LP6db: track 40.3 -> 34.5 mm
- net VCF_IN: track 13.1 -> 18.8 mm
- net -12VA: track 131.5 -> 136.2 mm, vias 4 -> 2
- net VCFCnt: track 70.5 -> 74.9 mm
- net Net-(C2-Pad1): track 17.2 -> 13.5 mm
- net Net-(Q2-B): track 9.03 -> 11.9 mm
- net LP18db: track 43.4 -> 40.9 mm, vias 0 -> 1
- net VCF_OUT: track 22.8 -> 25.2 mm
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Other:
- board text added: "12"
- board text added: "18"
- board text added: "6"
- board text added: "debugVCFSeparate Rev2. 2025/8/31"
- board text removed: "debugVCFSeparate 2025/8/11"
