File: SynthBoard/EG.kicad_sch (KiCad schematic)
At the start: 6 parts

Commit message: SynthBorad
デジタルも配置した
Parts:
- added C14: 0.1uF, Capacitor_SMD:C_0805_2012Metric_Pad1.18x1.45mm_HandSolder, symbol Device:C
- added C15, C21, C22: 0805B103J500NT, Capacitor_SMD:C_0805_2012Metric_Pad1.18x1.45mm_HandSolder, symbol Device:C
- added IC8: PIC16F13145-I/SO, Package_SO:SOIC-20W_7.5x12.8mm_P1.27mm, symbol SamacSys_Parts:PIC16F13145-I_P
- added J5: ICSP EG, Connector_PinHeader_2.54mm:PinHeader_1x05_P2.54mm_Vertical, symbol Connector_Generic:Conn_01x05
- added R106, R111, R122: 0805W8F1000T5E, Resistor_SMD:R_0805_2012Metric_Pad1.20x1.40mm_HandSolder, symbol Device:R
- added R109, R110: 0805W8F1002T5E, Resistor_SMD:R_0805_2012Metric_Pad1.20x1.40mm_HandSolder, symbol Device:R
- added R97: 0805W8F1001T5E, Resistor_SMD:R_0805_2012Metric_Pad1.20x1.40mm_HandSolder, symbol Device:R
- added U9: MCP6232-E_P, Package_SO:SOIC-8_3.9x4.9mm_P1.27mm, symbol Device:Opamp_Dual
Connections:
- net +5VD: now also C14.1, IC8.1 (VDD), J5.4 (Pin_4), R97.2, U9.8 (V+)
- net AccLv: now also IC8.6 (RC4)
- net AmpWave: now also IC8.14 (RC2)
- net Attack: now also IC8.7 (RC3)
- net Decay: now also IC8.8 (RC6)
- net GNDD: now also C14.2, C15.2, C21.2, C22.2, IC8.20 (VSS), J5.3 (Pin_3), U9.4 (V-)
- net Release: now also IC8.10 (RB7); no longer VR25.2 (WIPER)
- new net: R111.1, U9.1, U9.2 (-)
- new net: C15.1, R106.1, R97.1
- new net: R122.1, U9.6 (-), U9.7
- new net: C22.1, R110.2, U9.5 (+)
- new net: C21.1, R109.2, U9.3 (+)
- new net EnvAmp: R111.2
- new net EnvFlt: R122.2
- new net Gate: IC8.11 (RB6)
- new net ICSPCLK_EG: IC8.18 (RA1/ICSPCLK), J5.1 (Pin_1)
- new net ICSPDT_EG: IC8.19 (RA0/ICSPDAT), J5.2 (Pin_2)
- new net PWM_outAmp: IC8.15 (RC1), R109.1
- new net PWM_outFlt: IC8.3 (RA4), R110.1
- new net Sustain: IC8.9 (RC7), VR25.2 (WIPER)
- new net accAmp: IC8.12 (RB5)
- new net accFlt: IC8.13 (RB4)
- new net ~MCLR_EG: IC8.4 (~{MCLR}/VPP/RA3), J5.5 (Pin_5), R106.2
- no-connect marks 0 -> 4
Other:
- note added: "0.01uF"
- note added: "100"
- note added: "10K"
