File: SynthBoard/Power.kicad_sch (KiCad schematic)
At the start: 2 parts, among them J6 A_Power, J7 D_Power

Commit message: SynthBoard
部品をSMDにしてVCO+LFOを配置した
Parts:
- removed J7: D_Power, Connector_PinSocket_2.54mm:PinSocket_1x02_P2.54mm_Vertical, symbol Connector_Generic:Conn_01x02

Commit message: SynthBorad
デジタルも配置した
Parts:
- added J3: D_Power, Connector_PinSocket_2.54mm:PinSocket_1x02_P2.54mm_Vertical, symbol Connector_Generic:Conn_01x02
Connections:
- new net +5VD: J3.1 (Pin_1)
- new net GNDD: J3.2 (Pin_2)
