File: SynthBoard/SynthBoard.kicad_pcb (KiCad board)
At the start: 2 copper layers, 300 x 80 mm, 203 parts, among them IC1 AS321KTR-G1, IC2 AS321KTR-G1, IC4 AS321KTR-G1, IC5 V3340M, IC6 AS321KTR-G1, IC7 HEF4013BT,653, J1 Output, J10 AudioOut, J11 VCF_ResoWav, J4 Conn_01x03, J5 DigiConn, J6 A_Power, J7 Input, J8 AudioIn, J9 VCAEnv, Q1 2SC1623(RANGE:300-400), Q2 2SC1623(RANGE:300-400), Q3 2SA812, Q4 2SC1623(RANGE:300-400), Q6 2SA812, Q7 2SA812, Q8 2SA812, SW1 MFP_240, U1 TJM4558CDT, U2 LM13700, U3 Opamp_Dual, U4 Opamp_Dual, U5 LM13700, U6 Opamp_Dual, U8 LM13700

Commit message: SynthBorad
デジタルも配置した
Parts:
- removed J11: VCF_ResoWav, Connector_PinSocket_2.54mm:PinSocket_1x02_P2.54mm_Vertical
- added C12: 0.1uF, Capacitor_SMD:C_0805_2012Metric_Pad1.18x1.45mm_HandSolder, B.Cu at (63.0, 70.3)
- added C14: 0.1uF, Capacitor_SMD:C_0805_2012Metric_Pad1.18x1.45mm_HandSolder, B.Cu at (333.8, 73.1)
- added C15: 0805B103J500NT, Capacitor_SMD:C_0805_2012Metric_Pad1.18x1.45mm_HandSolder, F.Cu at (332.2, 53.7)
- added C16: 0805B103J500NT, Capacitor_SMD:C_0805_2012Metric_Pad1.18x1.45mm_HandSolder, F.Cu at (75.1, 49.3)
- added C17: 0805B103J500NT, Capacitor_SMD:C_0805_2012Metric_Pad1.18x1.45mm_HandSolder, F.Cu at (58.6, 43.8)
- added C18: 0805B103J500NT, Capacitor_SMD:C_0805_2012Metric_Pad1.18x1.45mm_HandSolder, F.Cu at (58.5, 50.9)
- added C19: 0805B103J500NT, Capacitor_SMD:C_0805_2012Metric_Pad1.18x1.45mm_HandSolder, F.Cu at (70.7, 49.4)
- added C21: 0805B103J500NT, Capacitor_SMD:C_0805_2012Metric_Pad1.18x1.45mm_HandSolder, F.Cu at (311.5, 53.2)
- added C22: 0805B103J500NT, Capacitor_SMD:C_0805_2012Metric_Pad1.18x1.45mm_HandSolder, F.Cu at (323.7, 53.5)
- added IC3: PIC16F15325-I/SL, Package_SO:SOIC-14_3.9x8.7mm_P1.27mm, B.Cu at (55.2, 70.3)
- added IC8: PIC16F13145-I/SO, Package_SO:SOIC-20W_7.5x12.8mm_P1.27mm, B.Cu at (324.7, 73.6)
- added J2: ICSP LFO, Connector_PinHeader_2.54mm:PinHeader_1x05_P2.54mm_Vertical, F.Cu at (81.0, 44.5)
- added J3: D_Power, Connector_PinSocket_2.54mm:PinSocket_1x02_P2.54mm_Vertical, F.Cu at (247.4, 116.6)
- added R100: 0805W8F1002T5E, Resistor_SMD:R_0805_2012Metric_Pad1.20x1.40mm_HandSolder, F.Cu at (58.5, 46.1)
- added R103: 0805W8F1002T5E, Resistor_SMD:R_0805_2012Metric_Pad1.20x1.40mm_HandSolder, F.Cu at (58.5, 48.5)
- added R105: 0805W8F1002T5E, Resistor_SMD:R_0805_2012Metric_Pad1.20x1.40mm_HandSolder, F.Cu at (70.5, 51.7)
- added R106: 0805W8F1000T5E, Resistor_SMD:R_0805_2012Metric_Pad1.20x1.40mm_HandSolder, F.Cu at (332.3, 51.4)
- added R109: 0805W8F1002T5E, Resistor_SMD:R_0805_2012Metric_Pad1.20x1.40mm_HandSolder, F.Cu at (311.5, 50.9)
- added R110: 0805W8F1002T5E, Resistor_SMD:R_0805_2012Metric_Pad1.20x1.40mm_HandSolder, F.Cu at (323.7, 51.2)
- added R111: 0805W8F1000T5E, Resistor_SMD:R_0805_2012Metric_Pad1.20x1.40mm_HandSolder, F.Cu at (311.5, 48.8)
- added R122: 0805W8F1000T5E, Resistor_SMD:R_0805_2012Metric_Pad1.20x1.40mm_HandSolder, F.Cu at (323.7, 48.9)
- added R97: 0805W8F1001T5E, Resistor_SMD:R_0805_2012Metric_Pad1.20x1.40mm_HandSolder, F.Cu at (332.2, 49.1)
- added R98: 0805W8F1001T5E, Resistor_SMD:R_0805_2012Metric_Pad1.20x1.40mm_HandSolder, F.Cu at (75.1, 51.6)
- added R99: 0805W8F1000T5E, Resistor_SMD:R_0805_2012Metric_Pad1.20x1.40mm_HandSolder, F.Cu at (79.1, 49.3)
- added U7: MCP6234T-E/SL, Package_SO:SOIC-14_3.9x8.7mm_P1.27mm, F.Cu at (64.5, 47.4)
- added U9: MCP6232-E_P, Package_SO:SOIC-8_3.9x4.9mm_P1.27mm, F.Cu at (317.6, 50.7)
- J1: value Output -> DigiInput; footprint Connector_PinSocket_2.54mm:PinSocket_2x06_P2.54mm_Vertical -> Connector_PinSocket_2.54mm:PinSocket_1x05_P2.54mm_Vertical
- J4: value Conn_01x03 -> VCOOut; footprint Connector_PinSocket_2.54mm:PinSocket_1x03_P2.54mm_Vertical -> Connector_PinSocket_2.54mm:PinSocket_2x07_P2.54mm_Vertical
- J5: value DigiConn -> ICSP EG; footprint Connector_PinSocket_2.54mm:PinSocket_2x10_P2.54mm_Vertical -> Connector_PinHeader_2.54mm:PinHeader_1x05_P2.54mm_Vertical
- J7: value Input -> LFO; footprint Connector_PinSocket_2.54mm:PinSocket_2x06_P2.54mm_Vertical -> Connector_PinSocket_2.54mm:PinSocket_2x03_P2.54mm_Vertical
- J8: value AudioIn -> VCFOut; footprint Connector_PinSocket_2.54mm:PinSocket_1x02_P2.54mm_Vertical -> Connector_PinSocket_2.54mm:PinSocket_2x02_P2.54mm_Vertical
- VR27: value 3362P-1-104LF -> 3362P-1-501LF
- moved J5 222.6 mm to (326.8, 43.9), turned to -90 degrees
- moved J7 118.8 mm to (69.5, 95.8)
- moved J4 108.9 mm to (153.1, 113.4)
- moved J1 106.0 mm to (271.4, 116.5), turned to -90 degrees
- moved J6 77.4 mm to (223.6, 116.5)
- moved Q2 49.2 mm to (64.5, 97.6)
- moved R13 46.6 mm to (64.7, 94.4), turned to 0 degrees
- moved J8 44.5 mm to (202.2, 114.8)
- moved R12 43.6 mm to (61.2, 95.4), turned to 90 degrees
- moved R39 14.6 mm to (102.8, 49.7)
- moved R41 14.6 mm to (102.8, 45.3)
- moved R42 14.6 mm to (107.0, 45.3)
- moved R38 14.6 mm to (102.8, 51.8)
- moved R40 14.6 mm to (102.8, 47.5)
- moved R43 14.6 mm to (107.0, 47.5)
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Connections:
- C3 pad 1: VCF_IN -> VCOWave
- J1 pad 1: VCOWave -> CV
- J1 pad 2: VCOWave -> Gate
- J1 pad 3: Vso -> accAmp
- J1 pad 4: Vso -> accFlt
- J1 pad 5: VPseparate -> GNDD
- J4 pad 1: Sine -> VCOWave
- J4 pad 2: Triangle -> VCOWave
- J4 pad 3: GNDA -> Vso
- J5 pad 1: Raw_Sine -> ICSPCLK_EG
- J5 pad 2: Raw_Sine -> ICSPDT_EG
- J5 pad 3: Raw_Triangle -> GNDD
- J5 pad 4: Raw_Triangle -> +5VD
- J5 pad 5: Rate -> ~MCLR_EG
- J7 pad 1: VCF_IN -> Sine
- J7 pad 2: VCF_IN -> Square
- J7 pad 3: FilterEnv -> Triangle
- J7 pad 4: FilterEnv -> Randum
- J7 pad 5: LFOSine -> GNDA
- J7 pad 6: LFOSine -> GNDA
- R1 pad 1: ResoWav -> VCF_ResoWav
- R214 pad 1: Env -> EnvFlt
- R52 pad 1: VCAEnv -> EnvAmp
- VR13 pad 3: FilterEnv -> EnvFlt
- VR25 pad 2: Release -> Sustain
Other:
- board size 300 x 80 mm -> 298 x 80 mm
