File: SynthBoard/VCA.kicad_sch (KiCad schematic)
At the start: 30 parts, among them IC2 AS321KTR-G1, J10 AudioOut, J8 AudioIn, J9 VCAEnv, Q6 2SA812, U3 Opamp_Dual, U8 LM13700

Commit message: SynthBorad
デジタルも配置した
Parts:
- removed J8: AudioIn, Connector_PinSocket_2.54mm:PinSocket_1x02_P2.54mm_Vertical, symbol Connector_Generic:Conn_01x02
- removed J9: VCAEnv, Connector_PinSocket_2.54mm:PinSocket_1x02_P2.54mm_Vertical, symbol Connector_Generic:Conn_01x02
Connections:
- net VCAEnv renamed EnvAmp
