File: SynthBoard_Right/VCO_waveform.kicad_sch (KiCad schematic)
At the start: 24 parts, among them IC6 AS321KTR-G1, IC7 HEF4013BT,653, Q1 2SC1623(RANGE:300-400)

Commit message: SynthBoard
Rightを配置済
Leftの配線ミスを修正
Connections:
- net +5VA: no longer VR3.1 (CCW)
- net GNDA: now also VR3.1 (CCW)
Changed lines of the file:
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@@
-	(wire
-		(pts
-			(xy 175.26 85.09) (xy 175.26 81.28)
-		)
-		(stroke
-			(width 0)
-			(type default)
-		)
-	)
 	(wire
 		(pts
@@
 	(wire
 		(pts
+			(xy 171.45 85.09) (xy 175.26 85.09)
+		)
+		(stroke
+			(width 0)
+			(type default)
+		)
+	)
+	(wire
+		(pts
 			(xy 189.23 87.63) (xy 193.04 87.63)
 		)
@@
 	(wire
 		(pts
+			(xy 175.26 85.09) (xy 175.26 93.98)
+		)
+		(stroke
+			(width 0)
+			(type default)
+		)
+	)
+	(wire
+		(pts
 			(xy 116.84 149.86) (xy 90.17 149.86)
 		)
@@
 		(pts
 			(xy 193.04 34.29) (xy 193.04 87.63)
-		)
-		(stroke
-			(width 0)
-			(type default)
-		)
-	)
-	(wire
-		(pts
-			(xy 171.45 85.09) (xy 175.26 85.09)
 		)
 		(stroke
@@
 	)
 	(symbol
-		(lib_id "power:+5VA")
-		(at 175.26 81.28 0)
+		(lib_id "power:GNDA")
+		(at 175.26 93.98 0)
 		(unit 1)
 		(exclude_from_sim no)
@@
 		(on_board yes)
 		(dnp no)
-		(property "Reference" "#PWR04"
-			(at 175.26 85.09 0)
-			(effects
-				(font
-					(size 1.27 1.27)
-				)
-				(hide yes)
-			)
-		)
-		(property "Value" "+5VA"
-			(at 175.26 76.2 0)
+		(property "Reference" "#PWR025"
+			(at 175.26 100.33 0)
+			(effects
+				(font
+					(size 1.27 1.27)
+				)
+				(hide yes)
+			)
+		)
+		(property "Value" "GNDA"
+			(at 170.434 95.504 0)
 			(effects
 				(font
@@
 		)
 		(property "Footprint" ""
-			(at 175.26 81.28 0)
+			(at 175.26 93.98 0)
 			(effects
 				(font
@@
 		)
 		(property "Datasheet" ""
-			(at 175.26 81.28 0)
-			(effects
-				(font
-					(size 1.27 1.27)
-				)
-				(hide yes)
-			)
-		)
-		(property "Description" "Power symbol creates a global label with name \"+5VA\""
-			(at 175.26 81.28 0)
+			(at 175.26 93.98 0)
+			(effects
+				(font
+					(size 1.27 1.27)
+				)
+				(hide yes)
+			)
+		)
+		(property "Description" "Power symbol creates a global label with name \"GNDA\" , analog ground"
+			(at 175.26 93.98 0)
 			(effects
 				(font
@@
 			(project "SynthBoard"
 				(path "/92765e2f-a998-485f-b610-76a9d5b50cba/54ae8d1b-caf5-4a85-9663-2a3f476f2243"
-					(reference "#PWR04")
+					(reference "#PWR025")
 					(unit 1)
 				)
