File: SynthBoard_Right/EG.kicad_sch (KiCad schematic)
At the start: 19 parts, among them IC8 PIC16F13145-I/SO, J5 ICSP EG, U9 MCP6232-E_P

Commit message: SynthBoard Right
配線ミスを修正
Other:
- note added: "1K"
Changed lines of the file:
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@@
 		)
 	)
-	(text "10K"
+	(text "1K"
 		(exclude_from_sim no)
 		(at 237.998 86.106 0)

Commit message: SynthBoard Right
Basic部品で更新まで
Parts:
- C15, C21, C22: value 0805B103J500NT -> CL21B103KBANNNC
Changed lines of the file:
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@@
 			)
 		)
-		(property "Value" "0805B103J500NT"
+		(property "Value" "CL21B103KBANNNC"
 			(at 219.964 101.346 0)
 			(effects
@@
 			)
 		)
-		(property "Value" "0805B103J500NT"
+		(property "Value" "CL21B103KBANNNC"
 			(at 143.256 99.06 0)
 			(effects
@@
 			)
 		)
-		(property "Value" "0805B103J500NT"
+		(property "Value" "CL21B103KBANNNC"
 			(at 143.256 73.66 0)
 			(effects
