File: SynthBoard_Right/VCA.kicad_sch (KiCad schematic)
At the start: 28 parts, among them IC2 AS321KTR-G1, J10 AudioOut, Q6 2SA812, U3 Opamp_Dual, U8 LM13700

Commit message: SynthBoard Right
配線ミスを修正
Parts:
- U3: value Opamp_Dual -> TJM4558CDT
Connections:
- net GNDA: now also VR14.1 (CCW); no longer VR14.3 (CW)
- net at C9.2, R70.2: now also VR14.3 (CW); no longer VR14.1 (CCW)
Other:
- moved on the sheet: J10, VR14
Changed lines of the file:
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@@
 	(text "GND"
 		(exclude_from_sim no)
-		(at 278.13 100.584 0)
+		(at 278.13 99.314 0)
 		(effects
 			(font
@@
 	(text "AudioOut"
 		(exclude_from_sim no)
-		(at 280.416 97.79 0)
+		(at 280.416 96.52 0)
 		(effects
 			(font
@@
 	)
 	(junction
-		(at 227.33 97.79)
+		(at 227.33 96.52)
 		(diameter 0)
 		(color 0 0 0 0)
@@
 	(wire
 		(pts
-			(xy 229.87 97.79) (xy 227.33 97.79)
+			(xy 229.87 96.52) (xy 227.33 96.52)
 		)
 		(stroke
@@
 	(wire
 		(pts
-			(xy 229.87 95.25) (xy 227.33 95.25)
+			(xy 229.87 99.06) (xy 227.33 99.06)
 		)
 		(stroke
@@
 	(wire
 		(pts
-			(xy 200.66 74.93) (xy 200.66 83.82)
+			(xy 224.79 96.52) (xy 227.33 96.52)
 		)
 		(stroke
@@
 	(wire
 		(pts
-			(xy 257.81 81.28) (xy 257.81 95.25)
+			(xy 200.66 74.93) (xy 200.66 83.82)
 		)
 		(stroke
@@
 	(wire
 		(pts
-			(xy 257.81 97.79) (xy 269.24 97.79)
-		)
-		(stroke
-			(width 0)
-			(type default)
-		)
-	)
-	(wire
-		(pts
 			(xy 116.84 78.74) (xy 119.38 78.74)
 		)
@@
 	(wire
 		(pts
-			(xy 265.43 100.33) (xy 265.43 104.14)
+			(xy 265.43 99.06) (xy 265.43 102.87)
 		)
 		(stroke
@@
 	(wire
 		(pts
+			(xy 257.81 81.28) (xy 257.81 93.98)
+		)
+		(stroke
+			(width 0)
+			(type default)
+		)
+	)
+	(wire
+		(pts
 			(xy 87.63 139.7) (xy 87.63 124.46)
 		)
@@
 	(wire
 		(pts
-			(xy 269.24 100.33) (xy 265.43 100.33)
+			(xy 269.24 99.06) (xy 265.43 99.06)
 		)
 		(stroke
@@
 	(wire
 		(pts
-			(xy 227.33 97.79) (xy 227.33 100.33)
+			(xy 224.79 96.52) (xy 224.79 107.95)
 		)
 		(stroke
@@
 	(wire
 		(pts
-			(xy 227.33 95.25) (xy 227.33 97.79)
+			(xy 227.33 99.06) (xy 227.33 96.52)
+		)
+		(stroke
+			(width 0)
+			(type default)
+		)
+	)
+	(wire
+		(pts
+			(xy 257.81 96.52) (xy 269.24 96.52)
 		)
 		(stroke
@@
 	(wire
 		(pts
-			(xy 69.85 69.85) (xy 69.85 81.28)
+			(xy 257.81 99.06) (xy 257.81 104.14)
 		)
 		(stroke
@@
 	(wire
 		(pts
-			(xy 104.14 151.13) (xy 104.14 154.94)
+			(xy 69.85 69.85) (xy 69.85 81.28)
 		)
 		(stroke
@@
 	(wire
 		(pts
-			(xy 134.62 137.16) (xy 139.7 137.16)
+			(xy 104.14 151.13) (xy 104.14 154.94)
 		)
 		(stroke
@@
 	(wire
 		(pts
-			(xy 163.83 105.41) (xy 163.83 107.95)
+			(xy 134.62 137.16) (xy 139.7 137.16)
 		)
 		(stroke
@@
 	(wire
 		(pts
-			(xy 257.81 100.33) (xy 257.81 104.14)
+			(xy 163.83 105.41) (xy 163.83 107.95)
 		)
 		(stroke
@@
 	(symbol
 		(lib_id "power:GNDA")
-		(at 265.43 104.14 0)
+		(at 265.43 102.87 0)
 		(unit 1)
 		(exclude_from_sim no)
@@
 		(fields_autoplaced yes)
 		(property "Reference" "#PWR0126"
-			(at 265.43 110.49 0)
+			(at 265.43 109.22 0)
 			(effects
 				(font
@@
 		)
 		(property "Value" "GNDA"
-			(at 265.43 109.22 0)
+			(at 265.43 107.95 0)
 			(effects
 				(font
@@
 		)
 		(property "Footprint" ""
-			(at 265.43 104.14 0)
+			(at 265.43 102.87 0)
 			(effects
 				(font
@@
 		)
 		(property "Datasheet" ""
-			(at 265.43 104.14 0)
+			(at 265.43 102.87 0)
 			(effects
 				(font
@@
 		)
 		(property "Description" "Power symbol creates a global label with name \"GNDA\" , analog ground"
-			(at 265.43 104.14 0)
+			(at 265.43 102.87 0)
 			(effects
 				(font
@@
 	(symbol
 		(lib_id "Connector_Generic:Conn_01x02")
-		(at 274.32 97.79 0)
+		(at 274.32 96.52 0)
 		(unit 1)
 		(exclude_from_sim no)
@@
 		(dnp no)
 		(property "Reference" "J10"
-			(at 269.748 92.202 0)
+			(at 269.748 90.932 0)
 			(effects
 				(font
@@
 		)
 		(property "Value" "AudioOut"
-			(at 269.748 94.742 0)
+			(at 269.748 93.472 0)
 			(effects
 				(font
@@
 		)
 		(property "Footprint" "Connector_PinHeader_2.54mm:PinHeader_1x02_P2.54mm_Vertical"
-			(at 274.32 97.79 0)
+			(at 274.32 96.52 0)
 			(effects
 				(font
@@
 		)
 		(property "Datasheet" "~"
-			(at 274.32 97.79 0)
+			(at 274.32 96.52 0)
 			(effects
 				(font
@@
 		)
 		(property "Description" "Generic connector, single row, 01x02, script generated (kicad-library-utils/schlib/autogen/connector/)"
-			(at 274.32 97.79 0)
+			(at 274.32 96.52 0)
 			(effects
 				(font
@@
 		)
 		(property "Sim.Library" ""
-			(at 274.32 97.79 0)
+			(at 274.32 96.52 0)
 			(effects
 				(font
@@
 		)
 		(property "Sim.Name" ""
-			(at 274.32 97.79 0)
+			(at 274.32 96.52 0)
 			(effects
 				(font
@@
 	(symbol
 		(lib_id "power:GNDA")
-		(at 227.33 100.33 0)
+		(at 224.79 107.95 0)
 		(unit 1)
 		(exclude_from_sim no)
@@
 		(on_board yes)
 		(dnp no)
-		(fields_autoplaced yes)
 		(property "Reference" "#PWR0123"
-			(at 227.33 106.68 0)
+			(at 224.79 114.3 0)
 			(effects
 				(font
@@
 		)
 		(property "Value" "GNDA"
-			(at 227.33 105.41 0)
+			(at 224.79 113.03 0)
 			(effects
 				(font
@@
 		)
 		(property "Footprint" ""
-			(at 227.33 100.33 0)
+			(at 224.79 107.95 0)
 			(effects
 				(font
@@
 		)
 		(property "Datasheet" ""
-			(at 227.33 100.33 0)
+			(at 224.79 107.95 0)
 			(effects
 				(font
@@
 		)
 		(property "Description" "Power symbol creates a global label with name \"GNDA\" , analog ground"
-			(at 227.33 100.33 0)
+			(at 224.79 107.95 0)
 			(effects
 				(font
@@
 			)
 		)
-		(property "Value" "Opamp_Dual"
+		(property "Value" "TJM4558CDT"
 			(at 76.2 147.32 0)
 			(effects
@@
 			)
 		)
-		(property "Value" "Opamp_Dual"
+		(property "Value" "TJM4558CDT"
 			(at 127 144.78 0)
 			(effects
@@
 	(symbol
 		(lib_id "SamacSys_Parts:RK09D117000B")
-		(at 257.81 95.25 0)
-		(mirror y)
+		(at 257.81 99.06 180)
 		(unit 1)
 		(exclude_from_sim no)
@@
 		(dnp no)
 		(property "Reference" "VR14"
-			(at 243.586 88.392 0)
+			(at 243.84 87.122 0)
 			(effects
 				(font
@@
 		)
 		(property "Value" "Volume 100KA"
-			(at 244.348 90.678 0)
+			(at 244.348 89.662 0)
 			(effects
 				(font
@@
 		)
 		(property "Footprint" "SamacSys_parts:RK09D117000B"
-			(at 233.68 190.17 0)
+			(at 233.68 4.14 0)
 			(effects
 				(font
@@
 		)
 		(property "Datasheet" "https://tech.alpsalpine.com/prod/j/html/potentiometer/rotarypotentiometers/rk09k/rk09d117000b.html"
-			(at 233.68 290.17 0)
+			(at 233.68 -95.86 0)
 			(effects
 				(font
@@
 		)
 		(property "Description" "9-inch insulated shaft snap-in type RK09K/RK09D series"
-			(at 257.81 95.25 0)
+			(at 257.81 99.06 0)
 			(effects
 				(font
@@
 		)
 		(property "Height" "30"
-			(at 233.68 490.17 0)
+			(at 233.68 -295.86 0)
 			(effects
 				(font
@@
 		)
 		(property "Manufacturer_Name" "ALPS Electric"
-			(at 233.68 590.17 0)
+			(at 233.68 -395.86 0)
 			(effects
 				(font
@@
 		)
 		(property "Manufacturer_Part_Number" "RK09D117000B"
-			(at 233.68 690.17 0)
+			(at 233.68 -495.86 0)
 			(effects
 				(font
@@
 		)
 		(property "Mouser Part Number" "688-RK09D117000B"
-			(at 233.68 790.17 0)
+			(at 233.68 -595.86 0)
 			(effects
 				(font
@@
 		)
 		(property "Mouser Price/Stock" "https://www.mouser.co.uk/ProductDetail/Alps-Alpine/RK09D117000B?qs=3cOf6TWd2rbc67829PEbEQ%3D%3D"
-			(at 233.68 890.17 0)
+			(at 233.68 -695.86 0)
 			(effects
 				(font
@@
 		)
 		(property "Arrow Part Number" ""
-			(at 233.68 990.17 0)
+			(at 233.68 -795.86 0)
 			(effects
 				(font
@@
 		)
 		(property "Arrow Price/Stock" ""
-			(at 233.68 1090.17 0)
+			(at 233.68 -895.86 0)
 			(effects
 				(font
@@
 			)
 		)
-		(property "Value" "Opamp_Dual"
+		(property "Value" "TJM4558CDT"
 			(at 201.93 133.3499 0)
 			(effects

Commit message: SynthBoard Right
Basic部品で更新まで
Parts:
- R52, R57, R66, R70: value 0805W8J0104T5E -> 0805W8F1003T5E
- R64: value 0805W8J0512T5E -> 0805W8F5101T5E
- U3: value TJM4558CDT -> TL072CDT
Changed lines of the file:
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@@
 			)
 		)
-		(property "Value" "0805W8J0104T5E"
+		(property "Value" "0805W8F1003T5E"
 			(at 76.2 121.92 90)
 			(effects
@@
 			)
 		)
-		(property "Value" "0805W8J0104T5E"
+		(property "Value" "0805W8F1003T5E"
 			(at 54.61 134.62 90)
 			(effects
@@
 			)
 		)
-		(property "Value" "0805W8J0512T5E"
+		(property "Value" "0805W8F5101T5E"
 			(at 138.43 88.646 0)
 			(effects
@@
 			)
 		)
-		(property "Value" "TJM4558CDT"
+		(property "Value" "TL072CDT"
 			(at 76.2 147.32 0)
 			(effects
@@
 			)
 		)
-		(property "Value" "0805W8J0104T5E"
+		(property "Value" "0805W8F1003T5E"
 			(at 154.94 88.646 0)
 			(effects
@@
 			)
 		)
-		(property "Value" "0805W8J0104T5E"
+		(property "Value" "0805W8F1003T5E"
 			(at 219.71 92.456 0)
 			(effects
@@
 			)
 		)
-		(property "Value" "TJM4558CDT"
+		(property "Value" "TL072CDT"
 			(at 127 144.78 0)
 			(effects
@@
 			)
 		)
-		(property "Value" "TJM4558CDT"
+		(property "Value" "TL072CDT"
 			(at 201.93 133.3499 0)
 			(effects

Commit message: MC2
まとめて登録
Parts:
- removed Q6: 2SA812, SamacSys_parts:SOT95P240X120-3N, symbol SamacSys_Parts:2SA812
- added Q4: 2SA1162-GR_F_, SamacSys_parts:1SS294LFT, symbol SamacSys_Parts:2SA1162-GR_F_
Connections:
- net at R65.2: now also Q4.1 (B)
- net at R68.1: now also Q4.3 (C)
- net at R61.2, U3.6 (-): now also Q4.2 (E)
Changed lines of the file:
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@@
 	)
 	(symbol
+		(lib_id "SamacSys_Parts:2SA1162-GR_F_")
+		(at 149.86 137.16 0)
+		(mirror x)
+		(unit 1)
+		(exclude_from_sim no)
+		(in_bom yes)
+		(on_board yes)
+		(dnp no)
+		(property "Reference" "Q4"
+			(at 163.83 138.4301 0)
+			(effects
+				(font
+					(size 1.27 1.27)
+				)
+				(justify left)
+			)
+		)
+		(property "Value" "2SA1162-GR_F_"
+			(at 163.83 135.8901 0)
+			(effects
+				(font
+					(size 1.27 1.27)
+				)
+				(justify left)
+			)
+		)
+		(property "Footprint" "SamacSys_parts:1SS294LFT"
+			(at 163.83 35.89 0)
+			(effects
+				(font
+					(size 1.27 1.27)
+				)
+				(justify left top)
+				(hide yes)
+			)
+		)
+		(property "Datasheet" "https://toshiba.semicon-storage.com/ap-en/product/bipolar-transistor/bipolar-transistor/detail.2SA1162.html"
+			(at 163.83 -64.11 0)
+			(effects
+				(font
+					(size 1.27 1.27)
+				)
+				(justify left top)
+				(hide yes)
+			)
+		)
+		(property "Description" "Transistor Toshiba 2SA1162-GR(F) PNP Bipolar Transistor, 0.15 A, 50 V, 3-Pin SC-59"
+			(at 149.86 137.16 0)
+			(effects
+				(font
+					(size 1.27 1.27)
+				)
+				(hide yes)
+			)
+		)
+		(property "Height" "1.4"
+			(at 163.83 -264.11 0)
+			(effects
+				(font
+					(size 1.27 1.27)
+				)
+				(justify left top)
+				(hide yes)
+			)
+		)
+		(property "Manufacturer_Name" "Toshiba"
+			(at 163.83 -364.11 0)
+			(effects
+				(font
+					(size 1.27 1.27)
+				)
+				(justify left top)
+				(hide yes)
+			)
+		)
+		(property "Manufacturer_Part_Number" "2SA1162-GR(F)"
+			(at 163.83 -464.11 0)
+			(effects
+				(font
+					(size 1.27 1.27)
+				)
+				(justify left top)
+				(hide yes)
+			)
+		)
+		(property "Mouser Part Number" ""
+			(at 163.83 -564.11 0)
+			(effects
+				(font
+					(size 1.27 1.27)
+				)
+				(justify left top)
+				(hide yes)
+			)
+		)
+		(property "Mouser Price/Stock" ""
+			(at 163.83 -664.11 0)
+			(effects
+				(font
+					(size 1.27 1.27)
+				)
+				(justify left top)
+				(hide yes)
+			)
+		)
+		(property "Arrow Part Number" ""
+			(at 163.83 -764.11 0)
+			(effects
+				(font
+					(size 1.27 1.27)
+				)
+				(justify left top)
+				(hide yes)
+			)
+		)
+		(property "Arrow Price/Stock" ""
+			(at 163.83 -864.11 0)
+			(effects
+				(font
+					(size 1.27 1.27)
+				)
+				(justify left top)
+				(hide yes)
+			)
+		)
+		(pin "1"
+		)
+		(pin "2"
+		)
+		(pin "3"
+		)
+		(instances
+			(project "SynthBoard"
+				(path "/92765e2f-a998-485f-b610-76a9d5b50cba/3e1fadc0-1ea8-431e-ae01-135c41be23af"
+					(reference "Q4")
+					(unit 1)
+				)
+			)
+		)
+	)
+	(symbol
 		(lib_id "SamacSys_Parts:AS321KTR-E1")
 		(at 163.83 81.28 0)
@@
 					(unit 1)
 				)
-			)
-		)
-	)
-	(symbol
-		(lib_id "SamacSys_Parts:2SA812")
-		(at 149.86 137.16 0)
-		(mirror x)
-		(unit 1)
-		(exclude_from_sim no)
-		(in_bom yes)
-		(on_board yes)
-		(dnp no)
-		(property "Reference" "Q6"
-			(at 163.83 138.4301 0)
-			(effects
-				(font
-					(size 1.27 1.27)
-				)
-				(justify left)
-			)
-		)
-		(property "Value" "2SA812"
-			(at 163.83 135.8901 0)
-			(effects
-				(font
-					(size 1.27 1.27)
-				)
-				(justify left)
-			)
-		)
-		(property "Footprint" "SamacSys_parts:SOT95P240X120-3N"
-			(at 163.83 35.89 0)
-			(effects
-				(font
-					(size 1.27 1.27)
-				)
-				(justify left top)
-				(hide yes)
-			)
-		)
-		(property "Datasheet" "https://4donline.ihs.com/images/VipMasterIC/IC/GSCC/GSCC-S-A0010612759/GSCC-S-A0010613804-1.pdf?hkey=EF798316E3902B6ED9A73243A3159BB0"
-			(at 163.83 -64.11 0)
-			(effects
-				(font
-					(size 1.27 1.27)
-				)
-				(justify left top)
-				(hide yes)
-			)
-		)
-		(property "Description" "Silicon Epitaxial Planar Transistor,Commplementary to 2SC1623.  High DC current gain:hFE=200typ. (VCE=-6.0V,IC=-1.0mA)  High Voltage: VCEO=-50V."
-			(at 149.86 137.16 0)
-			(effects
-				(font
-					(size 1.27 1.27)
-				)
-				(hide yes)
-			)
-		)
-		(property "Height" "1.2"
-			(at 163.83 -264.11 0)
-			(effects
-				(font
-					(size 1.27 1.27)
-				)
-				(justify left top)
-				(hide yes)
-			)
-		)
-		(property "Manufacturer_Name" "Galaxy"
-			(at 163.83 -364.11 0)
-			(effects
-				(font
-					(size 1.27 1.27)
-				)
-				(justify left top)
-				(hide yes)
-			)
-		)
-		(property "Manufacturer_Part_Number" "2SA812"
-			(at 163.83 -464.11 0)
-			(effects
-				(font
-					(size 1.27 1.27)
-				)
-				(justify left top)
-				(hide yes)
-			)
-		)
-		(property "Mouser Part Number" ""
-			(at 163.83 -564.11 0)
-			(effects
-				(font
-					(size 1.27 1.27)
-				)
-				(justify left top)
-				(hide yes)
-			)
-		)
-		(property "Mouser Price/Stock" ""
-			(at 163.83 -664.11 0)
-			(effects
-				(font
-					(size 1.27 1.27)
-				)
-				(justify left top)
-				(hide yes)
-			)
-		)
-		(property "Arrow Part Number" ""
-			(at 163.83 -764.11 0)
-			(effects
-				(font
-					(size 1.27 1.27)
-				)
-				(justify left top)
-				(hide yes)
-			)
-		)
-		(property "Arrow Price/Stock" ""
-			(at 163.83 -864.11 0)
-			(effects
-				(font
-					(size 1.27 1.27)
-				)
-				(justify left top)
-				(hide yes)
-			)
-		)
-		(pin "3"
-		)
-		(pin "1"
-		)
-		(pin "2"
-		)
-		(instances
-			(project "SynthBoard"
-				(path "/92765e2f-a998-485f-b610-76a9d5b50cba/3e1fadc0-1ea8-431e-ae01-135c41be23af"
-					(reference "Q6")
-					(unit 1)
-				)
