File: SynthBoard_Rotary/VCOBoardRev2/EG_POT.kicad_sch (KiCad schematic)
At the start: 18 parts, among them IC8 PIC16F13145-I_P, IC9 MCP6232T-E/SN

Commit message: MC2 Synth-Board Rotary
V0.2
U10:PIn4 -12Vに接続
IC4:Pin12,13 デフォルト12でジャンパーパッドを追加
R86:三角波をS2に未接続だったのを修正
S2,S3:スイッチ動作を上下入れ替え
VR9:右に2.5mm移動に伴い周辺回路の配置を変更
冗長な配線を修正
ビアを打った
Parts:
- C26, C27, C28: footprint Capacitor_THT:C_Disc_D3.4mm_W2.1mm_P2.50mm -> Capacitor_THT:C_Disc_D4.3mm_W1.9mm_P5.00mm
Changed lines of the file:
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@@
 			)
 		)
-		(property "Footprint" "Capacitor_THT:C_Disc_D3.4mm_W2.1mm_P2.50mm"
+		(property "Footprint" "Capacitor_THT:C_Disc_D4.3mm_W1.9mm_P5.00mm"
 			(at 140.6652 87.63 0)
 			(effects
@@
 			)
 		)
-		(property "Footprint" "Capacitor_THT:C_Disc_D3.4mm_W2.1mm_P2.50mm"
+		(property "Footprint" "Capacitor_THT:C_Disc_D4.3mm_W1.9mm_P5.00mm"
 			(at 162.2552 132.08 0)
 			(effects
@@
 			)
 		)
-		(property "Footprint" "Capacitor_THT:C_Disc_D3.4mm_W2.1mm_P2.50mm"
+		(property "Footprint" "Capacitor_THT:C_Disc_D4.3mm_W1.9mm_P5.00mm"
 			(at 209.2452 134.62 0)
 			(effects
