File: SynthBoard_Rotary/VCOBoardRev2/VCF.kicad_sch (KiCad schematic)
At the start: 28 parts, among them U2 LM13700, U3 LM13700

Commit message: MC2 Synth-Board Rotary
V0.2
U10:PIn4 -12Vに接続
IC4:Pin12,13 デフォルト12でジャンパーパッドを追加
R86:三角波をS2に未接続だったのを修正
S2,S3:スイッチ動作を上下入れ替え
VR9:右に2.5mm移動に伴い周辺回路の配置を変更
冗長な配線を修正
ビアを打った
Parts:
- C13, C14, C15, C16: footprint Capacitor_THT:C_Disc_D5.0mm_W2.5mm_P2.50mm -> Capacitor_THT:C_Disc_D5.0mm_W2.5mm_P5.00mm
Changed lines of the file:
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@@
 			)
 		)
-		(property "Footprint" "Capacitor_THT:C_Disc_D5.0mm_W2.5mm_P2.50mm"
+		(property "Footprint" "Capacitor_THT:C_Disc_D5.0mm_W2.5mm_P5.00mm"
 			(at 205.4352 91.44 0)
 			(effects
@@
 			)
 		)
-		(property "Footprint" "Capacitor_THT:C_Disc_D5.0mm_W2.5mm_P2.50mm"
+		(property "Footprint" "Capacitor_THT:C_Disc_D5.0mm_W2.5mm_P5.00mm"
 			(at 206.7052 46.99 0)
 			(effects
@@
 			)
 		)
-		(property "Footprint" "Capacitor_THT:C_Disc_D5.0mm_W2.5mm_P2.50mm"
+		(property "Footprint" "Capacitor_THT:C_Disc_D5.0mm_W2.5mm_P5.00mm"
 			(at 126.6952 46.99 0)
 			(effects
@@
 			)
 		)
-		(property "Footprint" "Capacitor_THT:C_Disc_D5.0mm_W2.5mm_P2.50mm"
+		(property "Footprint" "Capacitor_THT:C_Disc_D5.0mm_W2.5mm_P5.00mm"
 			(at 126.6952 91.44 0)
 			(effects
