File: SynthBoard_Rotary/VCOBoardRev2/VCOSeparate.kicad_pcb (KiCad board)
At the start: 2 copper layers, 250 x 100 mm, 228 parts, among them IC1 AS321KTR-E1, IC10 AS321KTR-E1, IC2 V3340M, IC3 AS321KTR-E1, IC4 4013, IC5 PIC16F15325-I_P, IC6 AS321KTR-E1, IC7 MCP6232T-E/SN, IC8 PIC16F13145-I_P, IC9 MCP6232T-E/SN, J1 VCOOut, J11 AudioOut, J12 LFO, J13 LFO DigitalInput, J2 VCOIn, J4 EnvOut, J5 EG DigitalInput, J7 A_Power, J8 VCF_ResoWav, J9 AudioIn, Q1 2SC3325-Y, Q2 2SA1162-GR_F_, Q3 2SA1162-GR_F_, Q4 2SC3325-Y, Q5 2SA1162-GR_F_, Q6 2SA1162-GR_F_, Q7 2SC3325-Y, U1 Opamp_Dual, U10 Opamp_Dual, U2 LM13700, U3 LM13700, U5 LM13700, U6 Opamp_Dual, U8 Opamp_Dual

Commit message: MC2 Synth-Board Rotary
V0.2
U10:PIn4 -12Vに接続
IC4:Pin12,13 デフォルト12でジャンパーパッドを追加
R86:三角波をS2に未接続だったのを修正
S2,S3:スイッチ動作を上下入れ替え
VR9:右に2.5mm移動に伴い周辺回路の配置を変更
冗長な配線を修正
ビアを打った
Parts:
- added JP1: SolderJumper_2_Bridged, Jumper:SolderJumper-2_P1.3mm_Bridged2Bar_RoundedPad1.0x1.5mm, F.Cu at (94.3, 119.9)
- added JP2: SolderJumper_2_Open, Jumper:SolderJumper-2_P1.3mm_Open_RoundedPad1.0x1.5mm, F.Cu at (94.3, 116.9)
- added R86: 18K, Resistor_THT:R_Axial_DIN0207_L6.3mm_D2.5mm_P2.54mm_Vertical, F.Cu at (120.0, 33.0)
- C13, C14, C15, C16: footprint Capacitor_THT:C_Disc_D5.0mm_W2.5mm_P2.50mm -> Capacitor_THT:C_Disc_D5.0mm_W2.5mm_P5.00mm
- C22, C23, C26, C27, C28, C31: footprint Capacitor_THT:C_Disc_D3.4mm_W2.1mm_P2.50mm -> Capacitor_THT:C_Disc_D4.3mm_W1.9mm_P5.00mm
- moved TM6 21.0 mm to (232.4, 54.6), turned to 90 degrees
- moved R107 11.8 mm to (256.8, 57.9)
- moved R19 11.3 mm to (121.5, 45.4), turned to 180 degrees
- moved R20 11.1 mm to (120.1, 36.4), turned to 0 degrees
- moved Q3 9.27 mm to (255.3, 53.8), turned to -90 degrees
- moved Q6 8.95 mm to (255.4, 61.6), turned to -90 degrees
- moved R81 7.61 mm to (251.2, 51.3)
- moved R85 7.61 mm to (251.2, 54.6)
- moved R101 6.57 mm to (247.9, 66.5), turned to 90 degrees
- moved R100 6.32 mm to (251.3, 66.5), turned to 90 degrees
- moved R104 4.14 mm to (251.2, 60.6), turned to 90 degrees
- moved R113 3.28 mm to (32.1, 120.2)
- moved C27 2.91 mm to (227.9, 117.9), turned to 180 degrees
- moved VR9 2.72 mm to (232.6, 46.0)
- moved R34 2.69 mm to (87.5, 119.5)
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Connections:
- IC4 pad 13: Net-(IC4A-C) -> Net-(IC4B-Q)
- R19 pad 2: Net-(S2-NC_3) -> Net-(S2-NC_1)
- R20 pad 1: LFO_Tri -> Net-(S2-NC_3)
- S2 pad 1: LFO_Tri -> Net-(S2-NC_1)
- S2 pad 4: LFO_Tri -> Net-(S2-NC_1)
- S3 pad 1: Sub1oct -> Sub2octPW
- S3 pad 3: Sub2octPW -> Sub1oct
- S3 pad 4: Sub1oct -> Sub2octPW
- S3 pad 6: Sub2octPW -> Sub1oct
- U10 pad 4: GNDA -> -12VA
Routing:
- net Triangle: track 20.9 -> 104.4 mm
- net -12VA: track 472.5 -> 517.9 mm
- net EG_GND: track 275.5 -> 255.6 mm, vias 12 -> 157
- net VCACnt: track 41.6 -> 56.1 mm, vias 0 -> 1
- net LFO_Tri: track 11.7 -> 0.00 mm
- net EnvFlt: track 177.6 -> 186.2 mm, vias 3 -> 5
- net Sub2octPW: track 32.4 -> 24.0 mm
- net Net-(S2-NC_1): track 0.00 -> 8.36 mm
- net +5VA: track 289.2 -> 297.3 mm, vias 3 -> 4
- net Sub1oct: track 32.3 -> 40.2 mm
- net Sub2oct: track 36.4 -> 28.9 mm
- net Net-(IC6-INPUT_-): track 132.3 -> 139.3 mm
- net Net-(IC4B-D): track 10.4 -> 14.9 mm
- net Net-(VR9-CW): track 15.0 -> 10.7 mm
- net Net-(IC4B-Q): track 0.00 -> 4.10 mm
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Other:
- board text added: "MC2 SynthBoard Ver0.2 2026/2/22"
- board text removed: "MC2 SynthBoard Ver0.1 2025/12/20"
